Commit message: new urdf, without rotations

File: src/ur5_description/urdf/ur5.urdf.xacro (robot description, xacro)
@@ -77,4 +77,5 @@
     <xacro:property name="forearm_radius" value="0.040" />    <!-- manually measured -->
     <xacro:property name="wrist_radius" value="0.045" />      <!-- manually measured -->
+    <!--mechanical structure of ur5 robot-->
     <link name="${prefix}base_link" >
       <visual>
@@ -314,5 +315,5 @@
       </collision>
       <xacro:cylinder_inertial radius="0.0375" length="0.0345" mass="${wrist_3_mass}">
-        <origin xyz="0.0 ${wrist_3_length - 0.0345/2} 0.0" rpy="${pi/2} 0 0" />
+        <origin xyz="0.0 ${wrist_3_length - 0.0345/2} 0.0" rpy="0 0 0" />
       </xacro:cylinder_inertial>
     </link>
@@ -322,4 +323,5 @@
       <origin xyz="0.0 ${wrist_3_length} 0.0" rpy="0.0 0.0 ${pi/2.0}" />
     </joint>
+    <!--end effector (link)-->
     <link name="${prefix}ee_link">
       <collision>
@@ -327,8 +329,10 @@
           <box size="0.01 0.01 0.01"/>
         </geometry>
-        <origin rpy="0 0 0" xyz="-0.01 0 0"/>
-      </collision>
-    </link>
+        <origin xyz="-0.01 0 0" rpy="0 0 0"/>
+      </collision>
+    </link>
+    <!--transmission interface of ur5 robot-->
     <xacro:ur_arm_transmission prefix="${prefix}" hw_interface="${transmission_hw_interface}" />
+    <!--gazebo configuration of ur5 robot-->
     <xacro:ur_arm_gazebo prefix="${prefix}" />
     <!-- ROS base_link to UR 'Base' Coordinates transform -->
@@ -343,5 +347,5 @@
       <child link="${prefix}base"/>
     </joint>
-    <!-- Frame coincident with all-zeros TCP on UR controller -->
+    <!-- Frame coincident with all-zeros TCP on UR controller
     <link name="${prefix}tool0"/>
     <joint name="${prefix}wrist_3_link-tool0_fixed_joint" type="fixed">
@@ -349,5 +353,5 @@
       <parent link="${prefix}wrist_3_link"/>
       <child link="${prefix}tool0"/>
-    </joint>
+    </joint> -->
   </xacro:macro>
 </robot>

File: src/ur5_description/urdf/ur5_joint_limited_robot.urdf (robot description, URDF)
Before this commit: robot ur5, 11 links, 10 joints
Links:
- removed link tool0
Joints:
- removed joint wrist_3_link-tool0_fixed_joint

Commit message: urdf from universal robot github

File: src/ur5_description/urdf/ur5.urdf.xacro (robot description, xacro)
@@ -77,5 +77,4 @@
     <xacro:property name="forearm_radius" value="0.040" />    <!-- manually measured -->
     <xacro:property name="wrist_radius" value="0.045" />      <!-- manually measured -->
-    <!--mechanical structure of ur5 robot-->
     <link name="${prefix}base_link" >
       <visual>
@@ -315,5 +314,5 @@
       </collision>
       <xacro:cylinder_inertial radius="0.0375" length="0.0345" mass="${wrist_3_mass}">
-        <origin xyz="0.0 ${wrist_3_length - 0.0345/2} 0.0" rpy="0 0 0" />
+        <origin xyz="0.0 ${wrist_3_length - 0.0345/2} 0.0" rpy="${pi/2} 0 0" />
       </xacro:cylinder_inertial>
     </link>
@@ -329,5 +328,5 @@
           <box size="0.01 0.01 0.01"/>
         </geometry>
-        <origin xyz="-0.01 0 0" rpy="0 0 0"/>
+        <origin rpy="0 0 0" xyz="-0.01 0 0"/>
       </collision>
     </link>
@@ -347,5 +346,5 @@
       <child link="${prefix}base"/>
     </joint>
-    <!-- Frame coincident with all-zeros TCP on UR controller
+    <!-- Frame coincident with all-zeros TCP on UR controller -->
     <link name="${prefix}tool0"/>
     <joint name="${prefix}wrist_3_link-tool0_fixed_joint" type="fixed">
@@ -353,5 +352,5 @@
       <parent link="${prefix}wrist_3_link"/>
       <child link="${prefix}tool0"/>
-    </joint> -->
+    </joint>
   </xacro:macro>
 </robot>
